Commit message: Port real-hardware perception pipeline: ground segmentation + multi-track predictor
Adds ground_segmentation/ground_segmentation_ros2 (vendored GSeg3D) as a
standalone node that splits the raw Livox cloud into ground/obstacle points,
replacing the pointcloud_to_laserscan-based front end for dynamic obstacle
detection. dynamic_obstacle_predictor now consumes obstacle_points
(PointCloud2) directly instead of /scan (LaserScan), with segmentation
retuned for the much denser point-per-object regime this produces
(segment_min_points raised, segment center now uses the full-segment
centroid instead of just the two angular extremes, plus a geometric/
kinematic hysteresis for the near-side/far-side disambiguation) to curb
spurious velocity on static objects.

PredictedPathObstacleLayer now reads /predicted_obstacle_markers
(MarkerArray, one path per active track) instead of the single-track
/predicted_obstacle_path, so the Nav2 costmap reflects every currently
tracked moving obstacle, not just the primary one.

Also includes the real-hardware URDF extrinsics (imu/lidar/camera frames
from bag /tf_static), bag_replay/robot_real/hardware_bringup launch files,
and local/global costmap sizing tuned for the real Livox range.

File: src/mrvk_description/urdf/camera_macro.urdf.xacro (robot description, xacro)
@@ -255,6 +255,6 @@
                           radius="${lens_radius}"
                           length="${lens_length}"
-                          xyz="${lens_x} ${lens_y} ${lens_z}"
-                          rpy="0.0 ${pitch} 0.0"
+                          xyz="0.167663 0.0 0.194112"
+                          rpy="-1.8288456 0.0022189 -1.5752228"
                           parent="${parent}"/>
         <!-- ========================================================= Links -->

File: src/mrvk_description/urdf/lidar_macro.urdf.xacro (robot description, xacro)
@@ -7,7 +7,7 @@
         <xacro:property name="size_y" value="0.03"/>
         <xacro:property name="size_z" value="0.04"/>
-        <xacro:property name="origin_x" value="0.20"/>
+        <xacro:property name="origin_x" value="0.207875"/>
         <xacro:property name="origin_y" value="0.0"/>
-        <xacro:property name="origin_z" value="0.09"/>
+        <xacro:property name="origin_z" value="0.128825"/>
         <!-- Link -->
         <link name="${name}">

File: src/mrvk_description/urdf/robot.plugins.xacro (robot description, xacro)
@@ -39,5 +39,5 @@
     </gazebo>
     <!-- ============================== IMU ============================== -->
-    <gazebo reference="imu_link">
+    <gazebo reference="imu_frame">
         <sensor name="imu_sensor" type="imu">
             <always_on>true</always_on>
@@ -60,5 +60,5 @@
                     <remapping>~/out:=/imu_data</remapping>
                 </ros>
-                <frame_name>imu_link</frame_name>
+                <frame_name>imu_frame</frame_name>
                 <initial_orientation_as_reference>false</initial_orientation_as_reference>
             </plugin>
@@ -66,5 +66,5 @@
     </gazebo>
     <!-- ================= Hokuyo URG-04LX Laser Range Finder ================= -->
-    <gazebo reference="sensor_laser_link">
+    <gazebo reference="lidar_frame">
         <sensor type="gpu_ray" name="head_hokuyo_sensor">
             <pose>0.0 0.0 0.0 0.0 0.0 0.0</pose>
@@ -96,10 +96,10 @@
                 </ros>
                 <output_type>sensor_msgs/LaserScan</output_type>
-                <frame_name>sensor_laser_link</frame_name>
+                <frame_name>lidar_frame</frame_name>
             </plugin>
         </sensor>
     </gazebo>
     <!-- ============================= Camera ============================= -->
-    <gazebo reference="camera_link">
+    <gazebo reference="camera_frame">
         <sensor type="camera" name="camera1">
             <update_rate>30.0</update_rate>
@@ -124,5 +124,5 @@
                 </ros>
                 <camera_name>camera</camera_name>
-                <frame_name>camera_link</frame_name>
+                <frame_name>camera_frame</frame_name>
                 <hack_baseline>0.07</hack_baseline>
             </plugin>

File: src/mrvk_description/urdf/robot.urdf.xacro (robot description, xacro)
@@ -33,9 +33,9 @@
         parent="base_link"/>
     <!-- IMU -->
-    <xacro:imu_macro name="imu_link" xyz="0.0 0.0 0.0" parent="base_link"/>
+    <xacro:imu_macro name="imu_frame" xyz="0.152755 -0.02226 0.158525" parent="base_link"/>
     <!-- LIDAR -->
-    <xacro:lidar_macro name="sensor_laser_link" parent="base_link"/>
+    <xacro:lidar_macro name="lidar_frame" parent="base_link"/>
     <!-- Camera -->
-    <xacro:camera_macro name="camera_link" parent="base_link"/>
+    <xacro:camera_macro name="camera_frame" parent="base_link"/>
     <!-- Ultrasonic sensors -->
     <xacro:ultrasonic_sensor_macro
